File: Board/4700AudioPlayer.sch (KiCad schematic (older format))
At the start: 30 parts, among them U1 74HC164, U10 74HC74, U11 74HC04, U12 74HC590, U13 23K256-I_SN, U14 74LS157, U15 74HC595, U16 23K256-I_SN, U2 74HC164, U3 74HC164, U4 74HC164, U5 74HC40103, U6 74HC40103, U7 74HC40103, U8 74HC40103, U9 74LS10

Commit message: [Wave] Fixed wrong assignments of 3V3 and GND
Connections:
- net +3V3: now also U5.16 (VCC), U5.3 (TE), U6.16 (VCC), U6.3 (TE), U7.16 (VCC), U7.3 (TE), U8.16 (VCC), U8.3 (TE); no longer U5.8 (GND), U6.8 (GND), U7.8 (GND), U8.8 (GND)
- net GND: now also U5.8 (GND), U6.8 (GND), U7.8 (GND), U8.8 (GND); no longer U5.16 (VCC), U5.3 (TE), U6.16 (VCC), U6.3 (TE), U7.16 (VCC), U7.3 (TE), U8.16 (VCC), U8.3 (TE)
Changed lines of the file:
@@
 U 1 1 60B805CB
 P 30450 3950
-F 0 "U8" V 30800 2700 50  0000 L CNN
-F 1 "74HC40103" V 30900 2700 50  0000 L CNN
+F 0 "U8" V 30800 4900 50  0000 L CNN
+F 1 "74HC40103" V 30900 4600 50  0000 L CNN
 F 2 "Package_SO:SOIC-16_3.9x9.9mm_P1.27mm" H 30500 2050 50  0001 C CNN
 F 3 "https://www.ti.com/lit/ds/symlink/cd74hc40103.pdf" H 30500 2050 50  0001 C CNN
@@
 $EndComp
 $Comp
-L power:+3V3 #PWR012
-U 1 1 60BAC5FF
-P 31750 3600
-F 0 "#PWR012" H 31750 3450 50  0001 C CNN
-F 1 "+3V3" H 31765 3773 50  0000 C CNN
-F 2 "" H 31750 3600 50  0001 C CNN
-F 3 "" H 31750 3600 50  0001 C CNN
-	1    31750 3600
-	1    0    0    -1
-$EndComp
-$Comp
 L power:GND #PWR08
 U 1 1 60BC890E
@@
 U 1 1 60BCFFA3
 P 27700 3950
-F 0 "U7" V 28050 2700 50  0000 L CNN
-F 1 "74HC40103" V 28150 2700 50  0000 L CNN
+F 0 "U7" V 28050 4900 50  0000 L CNN
+F 1 "74HC40103" V 28150 4600 50  0000 L CNN
 F 2 "Package_SO:SOIC-16_3.9x9.9mm_P1.27mm" H 27750 2050 50  0001 C CNN
 F 3 "https://www.ti.com/lit/ds/symlink/cd74hc40103.pdf" H 27750 2050 50  0001 C CNN
@@
 Wire Wire Line
 	27950 2550 27950 2600
-$Comp
-L power:GND #PWR015
-U 1 1 60BCFFC0
-P 26650 4250
-F 0 "#PWR015" H 26650 4000 50  0001 C CNN
-F 1 "GND" H 26655 4077 50  0000 C CNN
-F 2 "" H 26650 4250 50  0001 C CNN
-F 3 "" H 26650 4250 50  0001 C CNN
-	1    26650 4250
-	1    0    0    -1
-$EndComp
-Wire Wire Line
-	26650 3950 26650 4250
-$Comp
-L power:+3V3 #PWR011
-U 1 1 60BCFFCC
-P 29000 3700
-F 0 "#PWR011" H 29000 3550 50  0001 C CNN
-F 1 "+3V3" H 29015 3873 50  0000 C CNN
-F 2 "" H 29000 3700 50  0001 C CNN
-F 3 "" H 29000 3700 50  0001 C CNN
-	1    29000 3700
-	1    0    0    -1
-$EndComp
-Wire Wire Line
-	29000 3700 29000 3950
 $Comp
 L power:GND #PWR07
@@
 U 1 1 60BDB690
 P 24950 3950
-F 0 "U6" V 25300 2700 50  0000 L CNN
-F 1 "74HC40103" V 25400 2700 50  0000 L CNN
+F 0 "U6" V 25300 4900 50  0000 L CNN
+F 1 "74HC40103" V 25400 4600 50  0000 L CNN
 F 2 "Package_SO:SOIC-16_3.9x9.9mm_P1.27mm" H 25000 2050 50  0001 C CNN
 F 3 "https://www.ti.com/lit/ds/symlink/cd74hc40103.pdf" H 25000 2050 50  0001 C CNN
@@
 Wire Wire Line
 	25200 2550 25200 2600
-$Comp
-L power:GND #PWR014
-U 1 1 60BDB6AD
-P 23900 4250
-F 0 "#PWR014" H 23900 4000 50  0001 C CNN
-F 1 "GND" H 23905 4077 50  0000 C CNN
-F 2 "" H 23900 4250 50  0001 C CNN
-F 3 "" H 23900 4250 50  0001 C CNN
-	1    23900 4250
-	1    0    0    -1
-$EndComp
 Wire Wire Line
 	23950 3950 23900 3950
-Wire Wire Line
-	23900 3950 23900 4250
-$Comp
-L power:+3V3 #PWR010
-U 1 1 60BDB6B9
-P 26250 3700
-F 0 "#PWR010" H 26250 3550 50  0001 C CNN
-F 1 "+3V3" H 26265 3873 50  0000 C CNN
-F 2 "" H 26250 3700 50  0001 C CNN
-F 3 "" H 26250 3700 50  0001 C CNN
-	1    26250 3700
-	1    0    0    -1
-$EndComp
-Wire Wire Line
-	26250 3700 26250 3950
 $Comp
 L power:GND #PWR06
@@
 L power:GND #PWR013
 U 1 1 60BDB6F9
-P 21150 4250
-F 0 "#PWR013" H 21150 4000 50  0001 C CNN
-F 1 "GND" H 21155 4077 50  0000 C CNN
-F 2 "" H 21150 4250 50  0001 C CNN
-F 3 "" H 21150 4250 50  0001 C CNN
-	1    21150 4250
+P 23500 4250
+F 0 "#PWR013" H 23500 4000 50  0001 C CNN
+F 1 "GND" H 23505 4077 50  0000 C CNN
+F 2 "" H 23500 4250 50  0001 C CNN
+F 3 "" H 23500 4250 50  0001 C CNN
+	1    23500 4250
 	1    0    0    -1
 $EndComp
@@
 	21200 3950 21150 3950
 Wire Wire Line
-	21150 3950 21150 4250
+	23500 3950 23500 4250
 $Comp
 L power:GND #PWR05
@@
 	24500 4600 23700 4600
 Wire Wire Line
-	23500 3700 23500 3950
-$Comp
-L power:+3V3 #PWR09
-U 1 1 60BDB705
-P 23500 3700
-F 0 "#PWR09" H 23500 3550 50  0001 C CNN
-F 1 "+3V3" H 23515 3873 50  0000 C CNN
-F 2 "" H 23500 3700 50  0001 C CNN
-F 3 "" H 23500 3700 50  0001 C CNN
-	1    23500 3700
-	1    0    0    -1
-$EndComp
-Wire Wire Line
 	21750 4450 21750 4700
 Wire Wire Line
@@
 Wire Wire Line
 	21750 2550 21750 3450
-Wire Wire Line
-	22650 2950 22650 3450
 Wire Wire Line
 	21500 6600 21550 6600
@@
 	21850 1350 24600 1350
 Connection ~ 21850 1350
-$Comp
-L power:+3V3 #PWR?
-U 1 1 60EA1851
-P 22650 2950
-F 0 "#PWR?" H 22650 2800 50  0001 C CNN
-F 1 "+3V3" H 22665 3123 50  0000 C CNN
-F 2 "" H 22650 2950 50  0001 C CNN
-F 3 "" H 22650 2950 50  0001 C CNN
-	1    22650 2950
-	1    0    0    -1
-$EndComp
-Wire Wire Line
-	25400 2950 25400 3450
 Wire Wire Line
 	25500 3100 25500 3450
@@
 $EndComp
 Wire Wire Line
-	28150 2950 28150 3450
-Wire Wire Line
 	28250 3100 28250 3450
 $Comp
@@
 	1    0    0    -1
 $EndComp
-Wire Wire Line
-	30900 2950 30900 3450
 Wire Wire Line
 	31000 3100 31000 3450
@@
 $EndComp
 Wire Wire Line
-	20350 2750 21150 2750
+	20350 2750 21000 2750
 Wire Wire Line
 	22750 3100 22750 3450
@@
 U 1 1 60BDB6DC
 P 22200 3950
-F 0 "U5" V 22550 2700 50  0000 L CNN
-F 1 "74HC40103" V 22650 2700 50  0000 L CNN
+F 0 "U5" V 22550 4900 50  0000 L CNN
+F 1 "74HC40103" V 22650 4600 50  0000 L CNN
 F 2 "Package_SO:SOIC-16_3.9x9.9mm_P1.27mm" H 22250 2050 50  0001 C CNN
 F 3 "https://www.ti.com/lit/ds/symlink/cd74hc40103.pdf" H 22250 2050 50  0001 C CNN
@@
 $EndComp
 Wire Wire Line
-	31750 3600 31750 3950
-Wire Wire Line
 	31750 3950 31650 3950
-Wire Wire Line
-	29800 3450 29800 3400
 Wire Wire Line
 	28900 3950 29000 3950
@@
 Wire Wire Line
 	29200 4600 29200 3400
-$Comp
-L power:GND #PWR016
-U 1 1 60BB2F77
-P 29400 4250
-F 0 "#PWR016" H 29400 4000 50  0001 C CNN
-F 1 "GND" H 29405 4077 50  0000 C CNN
-F 2 "" H 29400 4250 50  0001 C CNN
-F 3 "" H 29400 4250 50  0001 C CNN
-	1    29400 4250
-	1    0    0    -1
-$EndComp
-Wire Wire Line
-	29400 3950 29400 4250
 Wire Wire Line
 	29450 3950 29400 3950
-Connection ~ 29400 3950
-Wire Wire Line
-	29800 3400 29400 3400
-Wire Wire Line
-	29400 3400 29400 3950
-Wire Wire Line
-	27050 3450 27050 3400
-Wire Wire Line
-	27050 3400 26650 3400
-Wire Wire Line
-	26650 3400 26650 3950
 Wire Wire Line
 	26650 3950 26700 3950
-Connection ~ 26650 3950
-Wire Wire Line
-	23900 3950 23900 3400
-Wire Wire Line
-	23900 3400 24300 3400
-Wire Wire Line
-	24300 3400 24300 3450
-Connection ~ 23900 3950
 Wire Wire Line
 	23050 3400 23050 3450
@@
 	21000 3300 21000 3450
 Wire Wire Line
-	22750 3100 21150 3100
-Wire Wire Line
-	21150 3100 21150 2750
+	22750 3100 21000 3100
 Connection ~ 22750 3100
 Wire Wire Line
@@
 Wire Wire Line
 	26150 3950 26250 3950
-Wire Wire Line
-	21550 3450 21550 3400
-Wire Wire Line
-	21550 3400 21150 3400
-Wire Wire Line
-	21150 3400 21150 3950
-Connection ~ 21150 3950
 Text Label 11150 2600 0    39   ~ 0
 0
@@
 	15550 4350 13150 4350
 Connection ~ 13150 4350
+Text Label 4300 8450 0    50   ~ 0
+ram_clk
+Wire Wire Line
+	4300 8450 5500 8450
+Wire Wire Line
+	4300 8550 5500 8550
+$Comp
+L power:GND #PWR014
+U 1 1 60BDB6AD
+P 26250 4250
+F 0 "#PWR014" H 26250 4000 50  0001 C CNN
+F 1 "GND" H 26255 4077 50  0000 C CNN
+F 2 "" H 26250 4250 50  0001 C CNN
+F 3 "" H 26250 4250 50  0001 C CNN
+	1    26250 4250
+	1    0    0    -1
+$EndComp
+Wire Wire Line
+	26250 3950 26250 4250
+$Comp
+L power:GND #PWR015
+U 1 1 60BCFFC0
+P 29000 4250
+F 0 "#PWR015" H 29000 4000 50  0001 C CNN
+F 1 "GND" H 29005 4077 50  0000 C CNN
+F 2 "" H 29000 4250 50  0001 C CNN
+F 3 "" H 29000 4250 50  0001 C CNN
+	1    29000 4250
+	1    0    0    -1
+$EndComp
+Wire Wire Line
+	29000 3950 29000 4250
+Wire Wire Line
+	31750 3950 31750 4250
+$Comp
+L power:GND #PWR016
+U 1 1 60BB2F77
+P 31750 4250
+F 0 "#PWR016" H 31750 4000 50  0001 C CNN
+F 1 "GND" H 31755 4077 50  0000 C CNN
+F 2 "" H 31750 4250 50  0001 C CNN
+F 3 "" H 31750 4250 50  0001 C CNN
+	1    31750 4250
+	1    0    0    -1
+$EndComp
+Text Label 4300 8550 0    50   ~ 0
+n_ram_clk
+Wire Wire Line
+	21550 3000 22650 3000
+Wire Wire Line
+	22650 3000 22650 3450
+Wire Wire Line
+	30900 2950 30900 3000
+Wire Wire Line
+	24300 3000 25400 3000
+Wire Wire Line
+	25400 2950 25400 3000
+Wire Wire Line
+	25400 3000 25400 3450
+Connection ~ 25400 3000
+Wire Wire Line
+	28150 2950 28150 3000
+Wire Wire Line
+	27050 3000 28150 3000
+Connection ~ 28150 3000
+Wire Wire Line
+	28150 3000 28150 3450
+Wire Wire Line
+	29400 3000 29800 3000
+Connection ~ 30900 3000
+Wire Wire Line
+	30900 3000 30900 3450
+Wire Wire Line
+	29400 3000 29400 3950
+Wire Wire Line
+	29800 3000 29800 3450
+Connection ~ 29800 3000
+Wire Wire Line
+	29800 3000 30900 3000
+Wire Wire Line
+	26650 3000 27050 3000
+Connection ~ 27050 3000
+Wire Wire Line
+	27050 3000 27050 3450
+Wire Wire Line
+	26650 3000 26650 3950
+Wire Wire Line
+	23900 3000 24300 3000
+Connection ~ 24300 3000
+Wire Wire Line
+	23900 3000 23900 3950
+Wire Wire Line
+	24300 3000 24300 3450
+Wire Wire Line
+	21000 3100 21000 2750
+Wire Wire Line
+	21150 3000 21550 3000
+Connection ~ 21550 3000
+Wire Wire Line
+	21550 3000 21550 3450
+Wire Wire Line
+	21150 3000 21150 3950
+Connection ~ 22650 3000
+Wire Wire Line
+	22650 2950 22650 3000
 Wire Bus Line
 	30350 6000 30350 6800
+$Comp
+L power:+3V3 #PWR?
+U 1 1 60EA1851
+P 22650 2950
+F 0 "#PWR?" H 22650 2800 50  0001 C CNN
+F 1 "+3V3" H 22665 3123 50  0000 C CNN
+F 2 "" H 22650 2950 50  0001 C CNN
+F 3 "" H 22650 2950 50  0001 C CNN
+	1    22650 2950
+	1    0    0    -1
+$EndComp
 $EndSCHEMATC

Commit message: [RAM] CS for init sequence
Parts:
- added U? (x2): 74LS10, symbol 74xx:74LS08
- added U?: 74HC590, symbol 74xx:74HC590
- added U? (x2): 74HC04, symbol 74xx:74HC04
Connections:
- net +3V3: now also U?.16 (VCC)
- net GND: now also U?.10 (DS), U?.14 (~OE), U?.8 (GND)
- net n_ram_clk: now also U?.13 (CPR), U?.2
- net n_ram_ready: now also U?.1, U?.2
- net n_reset: now also U?.1 (~PL), U?.1 (~PL), U?.1, U?.10 (~MRC)
- net ram_clk: now also U?.11 (CPC)
- net at U?.9 (Q7): no longer U?.10 (DS)
- net ram1_setup_clk renamed ram_setup_clk
- net ram_setup_clk: now also U?.3; no longer U?.2 (CP)
- net ram1_setup_data renamed ram_setup_data
- removed net ram1_setup_init: U?.1 (~PL), U?.1 (~PL), U?.1 (~PL)
- new net: U?.3, U?.5
- new net ram_init_cs: U?.6
- no-connect marks 13 -> 20
Other:
- moved on the sheet: U?, U?B

Commit message: [Wave] Switched to parallel data bus
Parts:
- removed U1, U2, U3, U4: 74HC164, symbol 74xx:74HC164
- removed U12: 74HC590, symbol 74xx:74HC590
- removed U13, U16: 23K256-I_SN, Package_SO:SOIC-8_3.9x4.9mm_P1.27mm, symbol My_Memory_RAM:23K256-I_SN
- removed U15: 74HC595, symbol 74xx:74HC595
- removed U9: 74LS10, symbol 74xx:74LS10
- removed U?: 74HC04, symbol 74xx:74HC04
- removed U? (x6): 74LS165, symbol 74xx:74LS165
- removed U?: 74LS10, symbol 74xx:74LS08
- added U?: 74HC40103, Package_SO:SOIC-16_3.9x9.9mm_P1.27mm, symbol My_74xx:74HC40103
- added U? (x5): 74LS574, symbol 74xx:74LS574
Connections:
- net labels added: header_shift_clk, playback_cntdown_clk, ram_out0, ram_out1, ram_out2, ram_out3, ram_out4, ram_out5, ram_out6, ram_out7, sample0, sample1, sample2, sample3, sample4, sample5, sample6, sample7
- net labels removed: current_sample, n_ram_select, ram2_setup_clk, ram2_setup_data, ram2_setup_init, ram_clk_out, ram_data_out, ram_select, ram_setup_clk, ram_setup_data
- wire segments 447 -> 347
- no-connect marks 20 -> 7
Other:
- note removed: "<"
- note removed: "Read / Write"
- note removed: "Seq. mode, no hold"
- note removed: "Write status reg."
- note removed: "todo: maybe\ncheck for zeros \nas well"
- moved on the sheet: U10A, U11B, U14, U5, U6, U7, U8, U?A, U?B, U?C, UA
